Commit message: Imported upstream version '2.5.4' of 'upstream'

File: urdf/camera/openni.gazebo.xacro (robot description, xacro)
@@ -18,7 +18,16 @@
   <xacro:macro name="openni_camera_gazebo_v0" params="name">
     <gazebo reference="${name}_color_frame">
-      <sensor type="depth" name="${name}_frame_sensor">
+      <xacro:if value="${gazebo_version == 'classic'}">
+        <xacro:property name="camera_type" value="depth"/>
+      </xacro:if>
+      <xacro:if value="${gazebo_version == 'gazebo'}">
+        <xacro:property name="camera_type" value="rgbd_camera"/>
+      </xacro:if>
+      <sensor type="${camera_type}" name="${name}_frame_sensor">
         <always_on>true</always_on>
+        <visualize>true</visualize>
         <update_rate>30.0</update_rate>
+        <topic>${name}</topic>
+        <gz_frame_id>${name}_color_frame</gz_frame_id>
         <camera>
           <horizontal_fov>${63.0*M_PI/180.0}</horizontal_fov>
@@ -40,18 +49,20 @@
           </distortion>
         </camera>
-        <plugin name="${name}_frame_controller" filename="libgazebo_ros_camera.so">
-          <camera_name>${name}</camera_name>
-          <ros>
-            <!-- <namespace>${name}</namespace>-->
-            <remapping>${name}/image_raw:=${name}/rgb/image_raw</remapping>
-            <remapping>${name}/camera_info:=${name}/rgb/camera_info</remapping>
-            <remapping>${name}/depth/image_raw:=${name}/depth/image_raw</remapping>
-            <remapping>${name}/depth/camera_info:=${name}/depth/camera_info</remapping>
-            <remapping>${name}/points:=${name}/depth/points</remapping>
-          </ros>
-          <frame_name>${name}_color_optical_frame</frame_name>
-          <min_depth>0.3</min_depth>
-          <max_depth>8.0</max_depth>
-        </plugin>
+        <xacro:if value="${gazebo_version == 'classic'}">
+          <plugin name="${name}_frame_controller" filename="libgazebo_ros_camera.so">
+            <camera_name>${name}</camera_name>
+            <ros>
+              <!-- <namespace>${name}</namespace>-->
+              <remapping>${name}/image_raw:=${name}/rgb/image_raw</remapping>
+              <remapping>${name}/camera_info:=${name}/rgb/camera_info</remapping>
+              <remapping>${name}/depth/image_raw:=${name}/depth/image_raw</remapping>
+              <remapping>${name}/depth/camera_info:=${name}/depth/camera_info</remapping>
+              <remapping>${name}/points:=${name}/depth/points</remapping>
+            </ros>
+            <frame_name>${name}_color_optical_frame</frame_name>
+            <min_depth>0.3</min_depth>
+            <max_depth>8.0</max_depth>
+          </plugin>
+        </xacro:if>
       </sensor>
     </gazebo>

File: urdf/camera/orbbec_astra.urdf.xacro (robot description, xacro)
@@ -35,5 +35,5 @@
         <origin xyz="0 0 0" rpy="0 0 0"/>
         <geometry>
-          <mesh filename="package://tiago_description/meshes/camera/xtion_pro_live/xtion_pro_live.dae" />
+          <mesh filename="package://pal_urdf_utils/meshes/camera/xtion_pro_live.dae" />
         </geometry>
         <material name="Grey">

File: urdf/camera/structure_sensor.gazebo.xacro (robot description, xacro)
@@ -14,101 +14,114 @@
 <robot xmlns:xacro="http://ros.org/wiki/xacro">
   <xacro:macro name="structure_sensor_rgbd_camera_gazebo" params="name">
+    <xacro:if value="${gazebo_version == 'classic'}">
+      <xacro:property name="camera_type" value="depth"/>
+    </xacro:if>
+    <xacro:if value="${gazebo_version == 'gazebo'}">
+      <xacro:property name="camera_type" value="rgbd_camera"/>
+    </xacro:if>
     <gazebo reference="${name}_link">
       <!-- IR + depth -->
-      <sensor type="depth" name="${name}_frame_sensor">
-        <always_on>true</always_on>
-        <update_rate>6.0</update_rate>
-        <camera>
-          <horizontal_fov>${58.0 * deg_to_rad}</horizontal_fov>
-          <image>
-            <format>R8G8B8</format>
-            <width>320</width>
-            <height>240</height>
-          </image>
-          <clip>
-            <near>0.45</near>
-            <far>10.0</far>
-          </clip>
-          <distortion>
-            <k1>0.0</k1>
-            <k2>0.0</k2>
-            <k3>0.0</k3>
-            <p1>0.0</p1>
-            <p2>0.0</p2>
-          </distortion>
-        </camera>
-        <plugin name="${name}_ir" filename="libgazebo_ros_camera.so">
-          <camera_name>${name}</camera_name>
-          <frame_name>${name}_optical_frame</frame_name>
-          <max_depth>10.0</max_depth>
-          <ros>
-            <namespace>${namespace}</namespace>
-            <remapping>${name}/image_raw:=${name}/ir/image_raw</remapping>
-            <remapping>${name}/camera_info:=${name}/ir/camera_info</remapping>
-            <remapping>${name}/image_raw/compressed:=${name}/ir/image_raw/compressed</remapping>
-            <remapping>${name}/image_raw/compressedDepth:=${name}/ir/image_raw/compressedDepth</remapping>
-            <remapping>${name}/image_raw/theora:=${name}/ir/image_raw/theora</remapping>
-            <remapping>${name}/points:=${name}/depth/points</remapping>
-            <qos>
-              <topic name="${name}/ir/image_raw">
-                <publisher>
-                  <reliability>best_effort</reliability>
-                  <durability>volatile</durability>
-                  <history depth="1">keep_last</history>
-                  <liveliness>automatic</liveliness>
-                </publisher>
-              </topic>
-              <topic name="${name}/ir/image_raw/compressed">
-                <publisher>
-                  <reliability>best_effort</reliability>
-                  <durability>volatile</durability>
-                  <history depth="1">keep_last</history>
-                  <liveliness>automatic</liveliness>
-                </publisher>
-              </topic>
-              <topic name="${name}/ir/image_raw/compressedDepth">
-                <publisher>
-                  <reliability>best_effort</reliability>
-                  <durability>volatile</durability>
-                  <history depth="1">keep_last</history>
-                  <liveliness>automatic</liveliness>
-                </publisher>
-              </topic>
-              <topic name="${name}/depth/image_raw">
-                <publisher>
-                  <reliability>best_effort</reliability>
-                  <durability>volatile</durability>
-                  <history depth="1">keep_last</history>
-                  <liveliness>automatic</liveliness>
-                </publisher>
-              </topic>
-              <topic name="${name}/depth/image_raw/compressed">
-                <publisher>
-                  <reliability>best_effort</reliability>
-                  <durability>volatile</durability>
-                  <history depth="1">keep_last</history>
-                  <liveliness>automatic</liveliness>
-                </publisher>
-              </topic>
-              <topic name="${name}/depth/image_raw/compressedDepth">
-                <publisher>
-                  <reliability>best_effort</reliability>
-                  <durability>volatile</durability>
-                  <history depth="1">keep_last</history>
-                  <liveliness>automatic</liveliness>
-                </publisher>
-              </topic>
-              <topic name="${name}/depth/points">
-                <publisher>
-                  <reliability>best_effort</reliability>
-                  <durability>volatile</durability>
-                  <history depth="1">keep_last</history>
-                  <liveliness>automatic</liveliness>
-                </publisher>
-              </topic>
-            </qos>
-          </ros>
-        </plugin>
-      </sensor>
+        <sensor type="${camera_type}" name="${name}_frame_sensor">
+          <always_on>true</always_on>
+          <update_rate>6.0</update_rate>
+          <gz_frame_id>${name}_optical_frame</gz_frame_id>
+          <always_on>1</always_on>
+          <update_rate>10</update_rate>
+          <visualize>0</visualize>
+          <topic>${name}</topic>
+          <camera>
+            <horizontal_fov>${58.0 * deg_to_rad}</horizontal_fov>
+            <image>
+              <format>R8G8B8</format>
+              <width>320</width>
+              <height>240</height>
+            </image>
+            <clip>
+              <near>0.45</near>
+              <far>10.0</far>
+            </clip>
+            <distortion>
+              <k1>0.0</k1>
+              <k2>0.0</k2>
+              <k3>0.0</k3>
+              <p1>0.0</p1>
+              <p2>0.0</p2>
+            </distortion>
+          </camera>
+          <xacro:if value="${gazebo_version == 'classic'}">
+            <plugin name="${name}_ir" filename="libgazebo_ros_camera.so">
+              <camera_name>${name}</camera_name>
+              <frame_name>${name}_optical_frame</frame_name>
+              <max_depth>10.0</max_depth>
+              <ros>
+                <namespace>${namespace}</namespace>
+                <remapping>${name}/image_raw:=${name}/ir/image_raw</remapping>
+                <remapping>${name}/camera_info:=${name}/ir/camera_info</remapping>
+                <remapping>${name}/image_raw/compressed:=${name}/ir/image_raw/compressed</remapping>
+                <remapping>${name}/image_raw/compressedDepth:=${name}/ir/image_raw/compressedDepth</remapping>
+                <remapping>${name}/image_raw/theora:=${name}/ir/image_raw/theora</remapping>
+                <remapping>${name}/points:=${name}/depth/points</remapping>
+                <qos>
+                  <topic name="${name}/ir/image_raw">
+                    <publisher>
+                      <reliability>best_effort</reliability>
+                      <durability>volatile</durability>
+                      <history depth="1">keep_last</history>
+                      <liveliness>automatic</liveliness>
+                    </publisher>
+                  </topic>
+                  <topic name="${name}/ir/image_raw/compressed">
+                    <publisher>
+                      <reliability>best_effort</reliability>
+                      <durability>volatile</durability>
+                      <history depth="1">keep_last</history>
+                      <liveliness>automatic</liveliness>
+                    </publisher>
+                  </topic>
+                  <topic name="${name}/ir/image_raw/compressedDepth">
+                    <publisher>
+                      <reliability>best_effort</reliability>
+                      <durability>volatile</durability>
+                      <history depth="1">keep_last</history>
+                      <liveliness>automatic</liveliness>
+                    </publisher>
+                  </topic>
+                  <topic name="${name}/depth/image_raw">
+                    <publisher>
+                      <reliability>best_effort</reliability>
+                      <durability>volatile</durability>
+                      <history depth="1">keep_last</history>
+                      <liveliness>automatic</liveliness>
+                    </publisher>
+                  </topic>
+                  <topic name="${name}/depth/image_raw/compressed">
+                    <publisher>
+                      <reliability>best_effort</reliability>
+                      <durability>volatile</durability>
+                      <history depth="1">keep_last</history>
+                      <liveliness>automatic</liveliness>
+                    </publisher>
+                  </topic>
+                  <topic name="${name}/depth/image_raw/compressedDepth">
+                    <publisher>
+                      <reliability>best_effort</reliability>
+                      <durability>volatile</durability>
+                      <history depth="1">keep_last</history>
+                      <liveliness>automatic</liveliness>
+                    </publisher>
+                  </topic>
+                  <topic name="${name}/depth/points">
+                    <publisher>
+                      <reliability>best_effort</reliability>
+                      <durability>volatile</durability>
+                      <history depth="1">keep_last</history>
+                      <liveliness>automatic</liveliness>
+                    </publisher>
+                  </topic>
+                </qos>
+              </ros>
+            </plugin>
+          </xacro:if>
+        </sensor>
     </gazebo>
   </xacro:macro>

File: urdf/camera/structure_sensor.urdf.xacro (robot description, xacro)
@@ -73,5 +73,5 @@
     <link name="${name}_depth_optical_frame"/>
     <!-- extensions -->
-    <xacro:structure_sensor_rgbd_camera_gazebo name="${name}" />
+    <xacro:structure_sensor_rgbd_camera_gazebo name="${name}"/>
   </xacro:macro>
 </robot>

File: urdf/camera/xtion_pro_live.urdf.xacro (robot description, xacro)
@@ -34,5 +34,5 @@
         <origin xyz="0 0 0" rpy="0 0 0"/>
         <geometry>
-          <mesh filename="package://tiago_description/meshes/camera/xtion_pro_live/xtion_pro_live.dae" />
+          <mesh filename="package://pal_urdf_utils/meshes/camera/xtion_pro_live.dae" />
         </geometry>
         <material name="Grey">

File: urdf/ft_sensors/schunk.urdf.xacro (robot description, xacro)
@@ -40,5 +40,5 @@
       <parent link="${parent}" />
       <child link="${name}_ft_link" />
-      <origin xyz="${0.0157*0.5 + 0.001525} 0 0" rpy="${90.0 * deg_to_rad} 0 ${90.0 * deg_to_rad}" />
+      <origin xyz="0 0 0" rpy="0 ${90.0 * deg_to_rad} 0" />
     </joint>
     <!-- FT tool -->
@@ -65,5 +65,5 @@
       <parent link="${name}_ft_link" />
       <child link="${name}_ft_tool_link" />
-      <origin xyz="0 0 ${0.0157*0.5 + 0.00975*0.5 - 0.001525}" rpy="${-90.0 * deg_to_rad} ${-90.0 * deg_to_rad} 0" />
+      <origin xyz="0 0 ${0.0157*0.5 + 0.00975*0.5 - 0.001525}" rpy="0 ${-90.0 * deg_to_rad} 0" />
     </joint>
     <!-- Gazebo config-->

File: urdf/interaction_sensors/imu.gazebo.xacro (robot description, xacro)
@@ -19,4 +19,5 @@
         <always_on>1</always_on>
         <update_rate>${update_rate}</update_rate>
+        <topic>${name}</topic>
         <imu>
           <noise>
@@ -36,11 +37,16 @@
           </noise>
         </imu>
-        <plugin name="${name}" filename="libgazebo_ros_imu_sensor.so">
-          <ros>
-            <namespace>${namespace}</namespace>
-            <!-- publish to /imu/data -->
-            <remapping>~/out:=${name}</remapping>
-          </ros>
-        </plugin>
+        <xacro:if value="${gazebo_version == 'classic'}">
+          <plugin name="${name}" filename="libgazebo_ros_imu_sensor.so">
+            <ros>
+              <namespace>${namespace}</namespace>
+              <!-- publish to /imu/data -->
+              <remapping>~/out:=${name}</remapping>
+            </ros>
+          </plugin>
+        </xacro:if>
+        <xacro:if value="${gazebo_version == 'gazebo'}">
+          <plugin filename="gz-sim-imu-system" name="gz::sim::systems::Imu"></plugin>
+        </xacro:if>
       </sensor>
     </gazebo>

File: urdf/interaction_sensors/imu_talos.gazebo.xacro (robot description, xacro)
@@ -15,24 +15,39 @@
   <xacro:macro name="imu_sensor_gazebo" params="update_rate">
     <gazebo reference="imu_link">
+        <gravity>true</gravity>
         <sensor name="imu_sensor" type="imu">
-        <always_on>1</always_on>
-        <update_rate>${update_rate}</update_rate>
-        <imu>
-            <noise>
-            <type>gaussian</type>
-            <rate>
-                <mean>0.0</mean>
-                <stddev>0.0</stddev>
-                <bias_mean>0.000000</bias_mean>
-                <bias_stddev>0.0000008</bias_stddev>
-            </rate>
-            <accel>
-                <mean>0.0</mean>
-                <stddev>0.0</stddev>
-                <bias_mean>0.0</bias_mean>
-                <bias_stddev>0.000</bias_stddev>
-            </accel>
-            </noise>
-        </imu>
+          <always_on>true</always_on>
+          <update_rate>${update_rate}</update_rate>
+          <topic>imu</topic>
+          <imu>
+              <noise>
+                <type>gaussian</type>
+                <rate>
+                    <mean>0.0</mean>
+                    <stddev>0.0</stddev>
+                    <bias_mean>0.000000</bias_mean>
+                    <bias_stddev>0.0000008</bias_stddev>
+                </rate>
+                <accel>
+                    <mean>0.0</mean>
+                    <stddev>0.0</stddev>
+                    <bias_mean>0.0</bias_mean>
+                    <bias_stddev>0.000</bias_stddev>
+                </accel>
+              </noise>
+              <initialOrientationAsReference>false</initialOrientationAsReference>
+          </imu>
+          <xacro:if value="${gazebo_version == 'classic'}">
+            <plugin name="gazebo_ros_imu_sensor" filename="libgazebo_ros_imu_sensor.so">
+              <ros>
+                <namespace>/talos</namespace>
+                <remapping>~/out:=imu</remapping>
+              </ros>
+              <initial_orientation_as_reference>false</initial_orientation_as_reference>
+            </plugin>
+          </xacro:if>
+          <xacro:if value="${gazebo_version == 'gazebo'}">
+            <plugin filename="gz-sim-imu-system" name="gz::sim::systems::Imu"></plugin>
+          </xacro:if>
         </sensor>
     </gazebo>

File: urdf/laser/hokuyo_urg_04lx_ug01_laser.gazebo.xacro (robot description, xacro)
@@ -15,8 +15,10 @@
   <xacro:macro name="hokuyo_urg_04lx_ug01_laser_gazebo" params="name ros_topic update_rate min_angle max_angle">
     <gazebo reference="${name}_link">
-      <sensor type="gpu_ray" name="${name}">
-        <pose>0 0 0 0 0 0</pose>
+      <sensor name="${name}" type="gpu_lidar">
         <update_rate>${update_rate}</update_rate>
+        <topic>${ros_topic}</topic>
+        <gz_frame_id>${name}_link</gz_frame_id>
         <visualize>true</visualize>
+        <always_on>true</always_on>
         <ray>
           <scan>
@@ -40,12 +42,19 @@
           </noise>
         </ray>
-        <plugin name="${name}" filename="libgazebo_ros_ray_sensor.so">
-          <ros>
-            <namespace>${namespace}</namespace>
-            <remapping>~/out:=${ros_topic}</remapping>
-          </ros>
-          <output_type>sensor_msgs/LaserScan</output_type>
-          <frame_name>${name}_link</frame_name>
-        </plugin>
+        <xacro:if value="${gazebo_version == 'classic'}">
+          <plugin name="${name}" filename="libgazebo_ros_ray_sensor.so">
+            <ros>
+              <namespace>${namespace}</namespace>
+              <remapping>~/out:=${ros_topic}</remapping>
+            </ros>
+            <output_type>sensor_msgs/LaserScan</output_type>
+            <frame_name>${name}_link</frame_name>
+          </plugin>
+        </xacro:if>
+        <xacro:if value="${gazebo_version == 'gazebo'}">
+          <plugin filename="gz-sim-sensors-system" name="gz::sim::systems::Sensors">
+            <render_engine>ogre2</render_engine>
+          </plugin>
+        </xacro:if>
       </sensor>
       <material>Gazebo/DarkGrey</material>

File: urdf/laser/range.gazebo.xacro (robot description, xacro)
@@ -15,8 +15,10 @@
   <xacro:macro name="range_gazebo" params="name ros_topic update_rate maxRange minRange fov radiation">
     <gazebo reference="${name}_link">
-      <sensor type="gpu_ray" name="${name}">
-        <pose>0 0 0 0 0 0</pose>
+      <sensor name="${name}" type="gpu_lidar">
         <update_rate>${update_rate}</update_rate>
+        <topic>${ros_topic}</topic>
+        <gz_frame_id>${name}_link</gz_frame_id>
         <visualize>false</visualize>
+        <always_on>true</always_on>
         <ray>
           <scan>
@@ -45,13 +47,20 @@
           </noise>
         </ray>
-        <plugin name="${name}_gazebo_ros_range" filename="libgazebo_ros_ray_sensor.so">
-          <ros>
-            <namespace>${namespace}</namespace>
-            <remapping>~/out:=${ros_topic}</remapping>
-          </ros>
-          <output_type>sensor_msgs/Range</output_type>
-          <radiation_type>${radiation}</radiation_type>
-          <frame_name>${name}_link</frame_name>
-        </plugin>
+        <xacro:if value="${gazebo_version == 'classic'}">
+          <plugin name="${name}_gazebo_ros_range" filename="libgazebo_ros_ray_sensor.so">
+            <ros>
+              <namespace>${namespace}</namespace>
+              <remapping>~/out:=${ros_topic}</remapping>
+            </ros>
+            <output_type>sensor_msgs/Range</output_type>
+            <radiation_type>${radiation}</radiation_type>
+            <frame_name>${name}_link</frame_name>
+          </plugin>
+        </xacro:if>
+        <xacro:if value="${gazebo_version == 'gazebo'}">
+          <!-- <plugin filename="gz-sim-sensors-system" name="gz::sim::systems::Sensors">
+            <render_engine>ogre2</render_engine>
+          </plugin> -->
+        </xacro:if>
       </sensor>
       <material>Gazebo/DarkGrey</material>

File: urdf/laser/sick_nanoscan3_laser.gazebo.xacro (robot description, xacro)
@@ -15,8 +15,10 @@
   <xacro:macro name="sick_nanoscan3_laser_gazebo" params="name ros_topic update_rate min_angle max_angle">
     <gazebo reference="${name}_link">
-      <sensor type="gpu_ray" name="${name}">
-        <pose>0 0 0 0 0 0</pose>
+      <sensor name="${name}" type="gpu_lidar">
         <update_rate>${update_rate}</update_rate>
+        <topic>${ros_topic}</topic>
+        <gz_frame_id>${name}_link</gz_frame_id>
         <visualize>true</visualize>
+        <always_on>true</always_on>
         <ray>
           <scan>
@@ -35,11 +37,18 @@
           </range>
         </ray>
-        <plugin filename="libgazebo_ros_laser.so" name="gazebo_ros_sick_laser">
-          <gaussianNoise>0.03</gaussianNoise>
-          <alwaysOn>true</alwaysOn>
-          <updateRate>${update_rate}</updateRate>
-          <topicName>${ros_topic}</topicName>
-          <frameName>${name}_link</frameName>
-        </plugin>
+        <xacro:if value="${gazebo_version == 'classic'}">
+          <plugin filename="libgazebo_ros_laser.so" name="gazebo_ros_sick_laser">
+            <gaussianNoise>0.03</gaussianNoise>
+            <alwaysOn>true</alwaysOn>
+            <updateRate>${update_rate}</updateRate>
+            <topicName>${ros_topic}</topicName>
+            <frameName>${name}_link</frameName>
+          </plugin>
+        </xacro:if>
+        <xacro:if value="${gazebo_version == 'gazebo'}">
+          <plugin filename="gz-sim-sensors-system" name="gz::sim::systems::Sensors">
+            <render_engine>ogre2</render_engine>
+          </plugin>
+        </xacro:if>
       </sensor>
       <material>Gazebo/DarkGrey</material>
