Commit message: Imported upstream version '2.5.4' of 'upstream'

File: urdf/laser/sick_tim551_laser.gazebo.xacro (robot description, xacro)
@@ -15,8 +15,10 @@
   <xacro:macro name="sick_tim551_laser_gazebo" params="name ros_topic update_rate min_angle max_angle">
     <gazebo reference="${name}_link">
-      <sensor type="gpu_ray" name="${name}">
-        <pose>0 0 0 0 0 0</pose>
+      <sensor name="${name}" type="gpu_lidar">
         <update_rate>${update_rate}</update_rate>
+        <topic>${ros_topic}</topic>
+        <gz_frame_id>${name}_link</gz_frame_id>
         <visualize>true</visualize>
+        <always_on>true</always_on>
         <ray>
           <scan>
@@ -40,12 +42,19 @@
           </noise>
         </ray>
-        <plugin name="${name}" filename="libgazebo_ros_ray_sensor.so">
-          <ros>
-            <namespace>${namespace}</namespace>
-            <remapping>~/out:=${ros_topic}</remapping>
-          </ros>
-          <output_type>sensor_msgs/LaserScan</output_type>
-          <frame_name>${name}_link</frame_name>
-        </plugin>
+        <xacro:if value="${gazebo_version == 'classic'}">
+          <plugin name="${name}" filename="libgazebo_ros_ray_sensor.so">
+            <ros>
+              <namespace>${namespace}</namespace>
+              <remapping>~/out:=${ros_topic}</remapping>
+            </ros>
+            <output_type>sensor_msgs/LaserScan</output_type>
+            <frame_name>${name}_link</frame_name>
+          </plugin>
+        </xacro:if>
+        <xacro:if value="${gazebo_version == 'gazebo'}">
+          <plugin filename="gz-sim-sensors-system" name="gz::sim::systems::Sensors">
+            <render_engine>ogre2</render_engine>
+          </plugin>
+        </xacro:if>
       </sensor>
       <material>Gazebo/DarkGrey</material>

File: urdf/laser/sick_tim561_laser.gazebo.xacro (robot description, xacro)
@@ -15,8 +15,10 @@
   <xacro:macro name="sick_tim561_laser_gazebo" params="name ros_topic update_rate min_angle max_angle">
     <gazebo reference="${name}_link">
-      <sensor type="gpu_ray" name="${name}">
-        <pose>0 0 0 0 0 0</pose>
+      <sensor name="${name}" type="gpu_lidar">
         <update_rate>${update_rate}</update_rate>
+        <topic>${ros_topic}</topic>
+        <gz_frame_id>${name}_link</gz_frame_id>
         <visualize>true</visualize>
+        <always_on>true</always_on>
         <ray>
           <scan>
@@ -40,12 +42,19 @@
           </noise>
         </ray>
-        <plugin name="${name}" filename="libgazebo_ros_ray_sensor.so">
-          <ros>
-            <namespace>${namespace}</namespace>
-            <remapping>~/out:=${ros_topic}</remapping>
-          </ros>
-          <output_type>sensor_msgs/LaserScan</output_type>
-          <frame_name>${name}_link</frame_name>
-        </plugin>
+        <xacro:if value="${gazebo_version == 'classic'}">
+          <plugin name="${name}" filename="libgazebo_ros_ray_sensor.so">
+            <ros>
+              <namespace>${namespace}</namespace>
+              <remapping>~/out:=${ros_topic}</remapping>
+            </ros>
+            <output_type>sensor_msgs/LaserScan</output_type>
+            <frame_name>${name}_link</frame_name>
+          </plugin>
+        </xacro:if>
+        <xacro:if value="${gazebo_version == 'gazebo'}">
+          <plugin filename="gz-sim-sensors-system" name="gz::sim::systems::Sensors">
+            <render_engine>ogre2</render_engine>
+          </plugin>
+        </xacro:if>
       </sensor>
       <material>Gazebo/DarkGrey</material>

File: urdf/laser/sick_tim571_laser.gazebo.xacro (robot description, xacro)
@@ -15,8 +15,10 @@
   <xacro:macro name="sick_tim571_laser_gazebo" params="name ros_topic update_rate min_angle max_angle">
     <gazebo reference="${name}_link">
-      <sensor type="gpu_ray" name="${name}">
-        <pose>0 0 0 0 0 0</pose>
+      <sensor name="${name}" type="gpu_lidar">
         <update_rate>${update_rate}</update_rate>
+        <topic>${ros_topic}</topic>
+        <gz_frame_id>${name}_link</gz_frame_id>
         <visualize>true</visualize>
+        <always_on>true</always_on>
         <ray>
           <scan>
@@ -25,5 +27,5 @@
               <samples>${818*(max_angle - min_angle)/(270.0 * deg_to_rad)}</samples>
               <resolution>1</resolution>              <!-- not the sensor resolution; just 1 -->
-              <min_angle>${min_angle}</min_angle>
+              <min_angle>${min_angle + deg_to_rad}</min_angle> <!--there is a laserscan detecting ghost obstacle-->
               <max_angle>${max_angle}</max_angle>
             </horizontal>
@@ -40,12 +42,19 @@
           </noise>
         </ray>
-        <plugin name="${name}" filename="libgazebo_ros_ray_sensor.so">
-          <ros>
-            <namespace>${namespace}</namespace>
-            <remapping>~/out:=${ros_topic}</remapping>
-          </ros>
-          <output_type>sensor_msgs/LaserScan</output_type>
-          <frame_name>${name}_link</frame_name>
-        </plugin>
+        <xacro:if value="${gazebo_version == 'classic'}">
+          <plugin name="${name}" filename="libgazebo_ros_ray_sensor.so">
+            <ros>
+              <namespace>${namespace}</namespace>
+              <remapping>~/out:=${ros_topic}</remapping>
+            </ros>
+            <output_type>sensor_msgs/LaserScan</output_type>
+            <frame_name>${name}_link</frame_name>
+          </plugin>
+        </xacro:if>
+        <xacro:if value="${gazebo_version == 'gazebo'}">
+          <plugin filename="gz-sim-sensors-system" name="gz::sim::systems::Sensors">
+            <render_engine>ogre2</render_engine>
+          </plugin>
+        </xacro:if>
       </sensor>
       <material>Gazebo/DarkGrey</material>

File: urdf/laser/sick_tim571_laser.urdf.xacro (robot description, xacro)
@@ -42,5 +42,5 @@
     </joint>
     <!-- gazebo extensions -->
-    <xacro:sick_tim571_laser_gazebo name="${name}" ros_topic="${ros_topic}" update_rate="${update_rate}" min_angle="${min_angle}" max_angle="${max_angle}" />
+    <xacro:sick_tim571_laser_gazebo name="${name}" ros_topic="${ros_topic}" update_rate="${update_rate}" min_angle="${min_angle}" max_angle="${max_angle}"/>
   </xacro:macro>
 </robot>

File: urdf/laser/ydlidar_tg15_laser.gazebo.xacro (robot description, xacro)
@@ -10,8 +10,10 @@
   <xacro:macro name="ydlidar_tg15_laser_gazebo" params="name ros_topic update_rate min_angle max_angle">
     <gazebo reference="${name}_link">
-      <sensor type="gpu_ray" name="${name}">
-        <pose>0 0 0 0 0 0</pose>
+      <sensor name="${name}" type="gpu_lidar">
         <update_rate>${update_rate}</update_rate>
+        <topic>${ros_topic}</topic>
+        <gz_frame_id>${name}_link</gz_frame_id>
         <visualize>true</visualize>
+        <always_on>true</always_on>
         <ray>
           <scan>
@@ -35,12 +37,19 @@
           </noise>
         </ray>
-        <plugin name="${name}" filename="libgazebo_ros_ray_sensor.so">
-            <ros>
-              <namespace>${namespace}</namespace>
-              <remapping>~/out:=${ros_topic}</remapping>
-            </ros>
-            <output_type>sensor_msgs/LaserScan</output_type>
-            <frame_name>${name}_link</frame_name>
-        </plugin>
+        <xacro:if value="${gazebo_version == 'classic'}">
+          <plugin name="${name}" filename="libgazebo_ros_ray_sensor.so">
+              <ros>
+                <namespace>${namespace}</namespace>
+                <remapping>~/out:=${ros_topic}</remapping>
+              </ros>
+              <output_type>sensor_msgs/LaserScan</output_type>
+              <frame_name>${name}_link</frame_name>
+          </plugin>
+        </xacro:if>
+        <xacro:if value="${gazebo_version == 'gazebo'}">
+          <plugin filename="gz-sim-sensors-system" name="gz::sim::systems::Sensors">
+            <render_engine>ogre2</render_engine>
+          </plugin>
+        </xacro:if>
       </sensor>
       <material>Gazebo/DarkGrey</material>

File: urdf/laser/ydlidar_tg30_laser.gazebo.xacro (robot description, xacro)
@@ -10,8 +10,10 @@
   <xacro:macro name="ydlidar_tg30_laser_gazebo" params="name ros_topic update_rate min_angle max_angle">
     <gazebo reference="${name}_link">
-      <sensor type="gpu_ray" name="${name}">
-        <pose>0 0 0 0 0 0</pose>
+      <sensor name="${name}" type="gpu_lidar">
         <update_rate>${update_rate}</update_rate>
+        <topic>${ros_topic}</topic>
+        <gz_frame_id>${name}_link</gz_frame_id>
         <visualize>true</visualize>
+        <always_on>true</always_on>
         <ray>
           <scan>
@@ -35,12 +37,19 @@
           </noise>
         </ray>
-        <plugin name="${name}" filename="libgazebo_ros_ray_sensor.so">
-            <ros>
-              <namespace>${namespace}</namespace>
-              <remapping>~/out:=${ros_topic}</remapping>
-            </ros>
-            <output_type>sensor_msgs/LaserScan</output_type>
-            <frame_name>${name}_link</frame_name>
-        </plugin>
+        <xacro:if value="${gazebo_version == 'classic'}">
+          <plugin name="${name}" filename="libgazebo_ros_ray_sensor.so">
+              <ros>
+                <namespace>${namespace}</namespace>
+                <remapping>~/out:=${ros_topic}</remapping>
+              </ros>
+              <output_type>sensor_msgs/LaserScan</output_type>
+              <frame_name>${name}_link</frame_name>
+          </plugin>
+        </xacro:if>
+        <xacro:if value="${gazebo_version == 'gazebo'}">
+          <plugin filename="gz-sim-sensors-system" name="gz::sim::systems::Sensors">
+            <render_engine>ogre2</render_engine>
+          </plugin>
+        </xacro:if>
       </sensor>
       <material>Gazebo/DarkGrey</material>

File: urdf/laser/ydlidar_tg30_laser.urdf.xacro (robot description, xacro)
@@ -21,5 +21,5 @@
         <origin xyz="0 0 0" rpy="0 0 0" />
         <geometry>
-          <mesh filename="package://pal_urdf_utils/meshes/laser/ydlidar.dae"/>
+          <mesh filename="package://pal_urdf_utils/meshes/laser/ydlidar.stl"/>
         </geometry>
         <material name="DarkGrey"/>
@@ -28,5 +28,5 @@
         <origin xyz="0 0 0" rpy="0 0 0" />
         <geometry>
-          <mesh filename="package://pal_urdf_utils/meshes/laser/ydlidar.dae"/>
+          <mesh filename="package://pal_urdf_utils/meshes/laser/ydlidar.stl"/>
         </geometry>
       </collision>
