Commit message: Imported upstream version '2.9.1' of 'upstream'

File: urdf/camera/realsense_d455.gazebo.xacro (robot description, xacro)
@@ -16,8 +16,18 @@
   <xacro:macro name="realsense_d455_rgbd_camera_gazebo" params="name" >
     <gazebo reference="${name}_link">
-      <sensor name="${name}" type="depth">
+      <xacro:if value="${gazebo_version == 'classic'}">
+        <xacro:property name="camera_type" value="depth"/>
+      </xacro:if>
+      <xacro:if value="${gazebo_version == 'gazebo'}">
+        <xacro:property name="camera_type" value="camera"/>
+      </xacro:if>
+      <sensor name="${name}" type="${camera_type}">
+        <xacro:if value="${gazebo_version == 'gazebo'}">
+          <topic>${name}/color</topic>
+          <gz_frame_id>${name}_depth_optical_frame</gz_frame_id>
+        </xacro:if>
         <camera name="${name}">
-          <horizontal_fov>${85.2*deg_to_rad}</horizontal_fov>
-          <vertical_fov>${58.0*deg_to_rad}</vertical_fov>
+          <horizontal_fov>${86.0*deg_to_rad}</horizontal_fov>
+          <vertical_fov>${57.0*deg_to_rad}</vertical_fov>
           <always_on>true</always_on>
           <update_rate>30</update_rate>
@@ -25,130 +35,151 @@
           <image>
             <format>B8G8R8</format>
-            <width>848</width>
+            <width>640</width>
             <height>480</height>
           </image>
-          <clip>
-            <near>0.3</near>
-            <far>3.0</far>
-          </clip>
-          <noise>
-            <type>gaussian</type>
-            <mean>0.0</mean>
-            <stddev>0.100</stddev>
-          </noise>
         </camera>
-        <plugin name="${name}" filename="libgazebo_ros_camera.so">
-          <frame_name>${name}_depth_optical_frame</frame_name>
-          <min_depth>0.1</min_depth>
-          <max_depth>10.0</max_depth>
-          <ros>
-            <namespace>${namespace}</namespace>
-            <remapping>${name}/image_raw:=${name}/color/image_raw</remapping>
-            <remapping>${name}/camera_info:=${name}/color/camera_info</remapping>
-            <remapping>${name}/image_raw/compressed:=${name}/color/image_raw/compressed</remapping>
-            <remapping>${name}/image_raw/compressedDepth:=${name}/color/image_raw/compressedDepth</remapping>
-            <remapping>${name}/image_raw/theora:=${name}/color/image_raw/theora</remapping>
-            <remapping>${name}/points:=${name}/depth/color/points</remapping>
-            <remapping>${name}/depth/image_raw:=${name}/depth/image_rect_raw</remapping>
-            <remapping>${name}/depth/image_raw/compressed:=${name}/depth/image_rect_raw/compressed</remapping>
-            <remapping>${name}/depth/image_raw/compressedDepth:=${name}/depth/image_rect_raw/compressedDepth</remapping>
-            <remapping>${name}/depth/image_raw/theora:=${name}/depth/image_rect_raw/theora</remapping>
-            <qos>
-              <topic name="${name}/color/image_raw">
-                <publisher>
-                  <reliability>best_effort</reliability>
-                  <durability>volatile</durability>
-                  <history depth="1">keep_last</history>
-                  <liveliness>automatic</liveliness>
-                </publisher>
-              </topic>
-              <topic name="${name}/color/camera_info">
-                <publisher>
-                  <reliability>best_effort</reliability>
-                  <durability>volatile</durability>
-                  <history depth="1">keep_last</history>
-                  <liveliness>automatic</liveliness>
-                </publisher>
-              </topic>
-              <topic name="${name}/color/image_raw/compressed">
-                <publisher>
-                  <reliability>best_effort</reliability>
-                  <durability>volatile</durability>
-                  <history depth="1">keep_last</history>
-                  <liveliness>automatic</liveliness>
-                </publisher>
-              </topic>
-              <topic name="${name}/color/image_raw/compressedDepth">
-                <publisher>
-                  <reliability>best_effort</reliability>
-                  <durability>volatile</durability>
-                  <history depth="1">keep_last</history>
-                  <liveliness>automatic</liveliness>
-                </publisher>
-              </topic>
-              <topic name="${name}/color/image_raw/theora">
-                <publisher>
-                  <reliability>best_effort</reliability>
-                  <durability>volatile</durability>
-                  <history depth="1">keep_last</history>
-                  <liveliness>automatic</liveliness>
-                </publisher>
-              </topic>
-              <topic name="${name}/depth/camera_info">
-                <publisher>
-                  <reliability>best_effort</reliability>
-                  <durability>volatile</durability>
-                  <history depth="1">keep_last</history>
-                  <liveliness>automatic</liveliness>
-                </publisher>
-              </topic>
-              <topic name="${name}/depth/color/points">
-                <publisher>
-                  <reliability>best_effort</reliability>
-                  <durability>volatile</durability>
-                  <history depth="1">keep_last</history>
-                  <liveliness>automatic</liveliness>
-                </publisher>
-              </topic>
-              <topic name="${name}/depth/image_rect_raw">
-                <publisher>
-                  <reliability>best_effort</reliability>
-                  <durability>volatile</durability>
-                  <history depth="1">keep_last</history>
-                  <liveliness>automatic</liveliness>
-                </publisher>
-              </topic>
-              <topic name="${name}/depth/image_rect_raw/compressed">
-                <publisher>
-                  <reliability>best_effort</reliability>
-                  <durability>volatile</durability>
-                  <history depth="1">keep_last</history>
-                  <liveliness>automatic</liveliness>
-                </publisher>
-              </topic>
-              <topic name="${name}/depth/image_rect_raw/compressedDepth">
-                <publisher>
-                  <reliability>best_effort</reliability>
-                  <durability>volatile</durability>
-                  <history depth="1">keep_last</history>
-                  <liveliness>automatic</liveliness>
-                </publisher>
-              </topic>
-              <topic name="${name}/depth/image_rect_raw/theora">
-                <publisher>
-                  <reliability>best_effort</reliability>
-                  <durability>volatile</durability>
-                  <history depth="1">keep_last</history>
-                  <liveliness>automatic</liveliness>
-                </publisher>
-              </topic>
-            </qos>
-          </ros>
-        </plugin>
+        <xacro:if value="${gazebo_version == 'classic'}">
+          <plugin name="${name}" filename="libgazebo_ros_camera.so">
+            <frame_name>${name}_depth_optical_frame</frame_name>
+            <min_depth>0.1</min_depth>
+            <max_depth>10.0</max_depth>
+            <ros>
+              <namespace>${namespace}</namespace>
+              <remapping>${name}/image_raw:=${name}/color/image_raw</remapping>
+              <remapping>${name}/camera_info:=${name}/color/camera_info</remapping>
+              <remapping>${name}/image_raw/compressed:=${name}/color/image_raw/compressed</remapping>
+              <remapping>${name}/image_raw/compressedDepth:=${name}/color/image_raw/compressedDepth</remapping>
+              <remapping>${name}/image_raw/theora:=${name}/color/image_raw/theora</remapping>
+              <remapping>${name}/points:=${name}/depth/color/points</remapping>
+              <remapping>${name}/depth/image_raw:=${name}/depth/image_rect_raw</remapping>
+              <remapping>${name}/depth/image_raw/compressed:=${name}/depth/image_rect_raw/compressed</remapping>
+              <remapping>${name}/depth/image_raw/compressedDepth:=${name}/depth/image_rect_raw/compressedDepth</remapping>
+              <remapping>${name}/depth/image_raw/theora:=${name}/depth/image_rect_raw/theora</remapping>
+              <qos>
+                <topic name="${name}/color/image_raw">
+                  <publisher>
+                    <reliability>best_effort</reliability>
+                    <durability>volatile</durability>
+                    <history depth="1">keep_last</history>
+                    <liveliness>automatic</liveliness>
+                  </publisher>
+                </topic>
+                <topic name="${name}/color/camera_info">
+                  <publisher>
+                    <reliability>best_effort</reliability>
+                    <durability>volatile</durability>
+                    <history depth="1">keep_last</history>
+                    <liveliness>automatic</liveliness>
+                  </publisher>
+                </topic>
+                <topic name="${name}/color/image_raw/compressed">
+                  <publisher>
+                    <reliability>best_effort</reliability>
+                    <durability>volatile</durability>
+                    <history depth="1">keep_last</history>
+                    <liveliness>automatic</liveliness>
+                  </publisher>
+                </topic>
+                <topic name="${name}/color/image_raw/compressedDepth">
+                  <publisher>
+                    <reliability>best_effort</reliability>
+                    <durability>volatile</durability>
+                    <history depth="1">keep_last</history>
+                    <liveliness>automatic</liveliness>
+                  </publisher>
+                </topic>
+                <topic name="${name}/color/image_raw/theora">
+                  <publisher>
+                    <reliability>best_effort</reliability>
+                    <durability>volatile</durability>
+                    <history depth="1">keep_last</history>
+                    <liveliness>automatic</liveliness>
+                  </publisher>
+                </topic>
+                <topic name="${name}/depth/camera_info">
+                  <publisher>
+                    <reliability>best_effort</reliability>
+                    <durability>volatile</durability>
+                    <history depth="1">keep_last</history>
+                    <liveliness>automatic</liveliness>
+                  </publisher>
+                </topic>
+                <topic name="${name}/depth/color/points">
+                  <publisher>
+                    <reliability>best_effort</reliability>
+                    <durability>volatile</durability>
+                    <history depth="1">keep_last</history>
+                    <liveliness>automatic</liveliness>
+                  </publisher>
+                </topic>
+                <topic name="${name}/depth/image_rect_raw">
+                  <publisher>
+                    <reliability>best_effort</reliability>
+                    <durability>volatile</durability>
+                    <history depth="1">keep_last</history>
+                    <liveliness>automatic</liveliness>
+                  </publisher>
+                </topic>
+                <topic name="${name}/depth/image_rect_raw/compressed">
+                  <publisher>
+                    <reliability>best_effort</reliability>
+                    <durability>volatile</durability>
+                    <history depth="1">keep_last</history>
+                    <liveliness>automatic</liveliness>
+                  </publisher>
+                </topic>
+                <topic name="${name}/depth/image_rect_raw/compressedDepth">
+                  <publisher>
+                    <reliability>best_effort</reliability>
+                    <durability>volatile</durability>
+                    <history depth="1">keep_last</history>
+                    <liveliness>automatic</liveliness>
+                  </publisher>
+                </topic>
+                <topic name="${name}/depth/image_rect_raw/theora">
+                  <publisher>
+                    <reliability>best_effort</reliability>
+                    <durability>volatile</durability>
+                    <history depth="1">keep_last</history>
+                    <liveliness>automatic</liveliness>
+                  </publisher>
+                </topic>
+              </qos>
+            </ros>
+          </plugin>
+        </xacro:if>
       </sensor>
+      <xacro:if value="${gazebo_version == 'gazebo'}">
+        <sensor name="${name}_frame_depth_sensor" type="rgbd_camera">
+          <always_on>1</always_on>
+          <gz_frame_id>${name}_depth_frame</gz_frame_id>
+          <update_rate>30.0</update_rate>
+          <visualize>1</visualize>
+          <topic>${name}/depth</topic>
+          <camera name="rgbd_camera_frame">
+            <horizontal_fov>${86.0*deg_to_rad}</horizontal_fov>
+            <vertical_fov>${57.0*deg_to_rad}</vertical_fov>
+            <image>
+              <width>640</width>
+              <height>480</height>
+              <format>B8G8R8</format>
+            </image>
+            <depth_camera>
+              <clip>
+                <near>0.6</near>
+                <far>6.0</far>
+              </clip>
+            </depth_camera>
+          </camera>
+        </sensor>
+      </xacro:if>
       <!-- IMU Sensor -->
       <sensor name="${name}_imu_sensor" type="imu">
         <always_on>1</always_on>
         <update_rate>200</update_rate>
+        <xacro:if value="${gazebo_version == 'gazebo'}">
+          <topic>${name}/imu</topic>
+          <gz_frame_id>${name}_imu_optical_frame</gz_frame_id>
+        </xacro:if>
         <imu>
           <noise>
@@ -168,22 +199,25 @@
           </noise>
         </imu>
-        <plugin name="${name}_imu" filename="libgazebo_ros_imu_sensor.so">
-          <frame_name>${name}_imu_optical_frame</frame_name>
-          <ros>
-            <namespace>${namespace}</namespace>
-            <!-- publish to /imu/data -->
-            <remapping>~/out:=${name}/imu</remapping>
-            <qos>
-              <topic name="${name}/imu">
-                <publisher>
-                  <reliability>best_effort</reliability>
-                  <durability>volatile</durability>
-                  <history depth="1">keep_last</history>
-                  <liveliness>automatic</liveliness>
-                </publisher>
-              </topic>
-            </qos>
-          </ros>
-        </plugin>
+        <xacro:if value="${gazebo_version == 'classic'}">
+          <plugin name="${name}_imu" filename="libgazebo_ros_imu_sensor.so">
+            <frame_name>${name}_imu_optical_frame</frame_name>
+            <ros>
+              <namespace>${namespace}</namespace>
+              <!-- publish to /imu/data -->
+              <remapping>~/out:=${name}/imu</remapping>
+              <qos>
+                <topic name="${name}/imu">
+                  <publisher>
+                    <reliability>best_effort</reliability>
+                    <durability>volatile</durability>
+                    <history depth="1">keep_last</history>
+                    <liveliness>automatic</liveliness>
+                  </publisher>
+                </topic>
+              </qos>
+            </ros>
+            <initial_orientation_as_reference>false</initial_orientation_as_reference>
+          </plugin>
+        </xacro:if>
       </sensor>
     </gazebo>

File: urdf/laser/sick_picoscan150core_laser.gazebo.xacro (robot description, xacro)
@@ -1,5 +1,5 @@
 <?xml version="1.0"?>
 <!--
-  Copyright (c) 2025 PAL Robotics S.L. All rights reserved.
+  Copyright (c) 2026 PAL Robotics S.L. All rights reserved.
   Licensed under the Apache License, Version 2.0 (the "License");
   you may not use this file except in compliance with the License.
@@ -13,5 +13,5 @@
  -->
 <robot xmlns:xacro="http://ros.org/wiki/xacro">
-  <xacro:macro name="sick_tim571_laser_gazebo" params="name ros_topic update_rate min_angle max_angle">
+  <xacro:macro name="sick_picoscan150core_laser_gazebo" params="name ros_topic update_rate min_angle max_angle">
     <gazebo reference="${name}_link">
       <sensor name="${name}" type="gpu_lidar">
@@ -24,6 +24,6 @@
           <scan>
             <horizontal>
-              <!-- 818 (270/0.33) steps in 270deg fov -->
-              <samples>${818*(max_angle - min_angle)/(270.0 * deg_to_rad)}</samples>
+              <!-- 1104 (276/0.25) steps in 276 deg fov -->
+              <samples>${1104*(max_angle - min_angle)/(276.0 * deg_to_rad)}</samples>
               <resolution>1</resolution>              <!-- not the sensor resolution; just 1 -->
               <min_angle>${min_angle + deg_to_rad}</min_angle> <!--there is a laserscan detecting ghost obstacle-->
@@ -34,5 +34,5 @@
             <min>0.05</min>
             <max>25.0</max>
-            <resolution>0.001</resolution>
+            <resolution>0.25</resolution>
           </range>
           <noise>
@@ -55,4 +55,38 @@
       <material>Gazebo/DarkGrey</material>
     </gazebo>
+    <gazebo reference="${name}_imu_link">
+      <sensor name="${name}_imu_sensor" type="imu">
+        <always_on>1</always_on>
+        <update_rate>100</update_rate>
+        <topic>${ros_topic}/imu</topic>
+        <imu>
+          <noise>
+            <type>gaussian</type>
+            <rate>
+              <mean>0.0</mean>
+              <stddev>2e-4</stddev>
+              <bias_mean>0.0000075</bias_mean>
+              <bias_stddev>0.0000008</bias_stddev>
+            </rate>
+            <accel>
+              <mean>0.0</mean>
+              <stddev>1.7e-2</stddev>
+              <bias_mean>0.1</bias_mean>
+              <bias_stddev>0.001</bias_stddev>
+            </accel>
+          </noise>
+        </imu>
+        <xacro:if value="${gazebo_version == 'classic'}">
+          <plugin name="${name}_imu_sensor" filename="libgazebo_ros_imu_sensor.so">
+            <ros>
+              <namespace>${namespace}</namespace>
+              <!-- publish to /imu/data -->
+              <remapping>~/out:=${ros_topic}/imu</remapping>
+            </ros>
+            <initial_orientation_as_reference>false</initial_orientation_as_reference>
+          </plugin>
+        </xacro:if>
+      </sensor>
+    </gazebo>
   </xacro:macro>
 </robot>
